File: PROYEK_BMS_NUVOTON.kicad_pcb (KiCad board)
At the start: 2 copper layers, 95.9 x 107.3 mm, 256 parts, among them J1 Conn_01x23_Pin, J2 Conn_01x04_Pin, J3 USB_B_Micro, J4 Screw_Terminal_01x02, Q1 NPN, Q10 Q_NMOS_GSD, Q11 Q_NMOS_GSD, Q12 Q_NMOS_GSD, Q13 Q_NMOS_GSD, Q14 Q_NMOS_GSD, Q15 Q_NMOS_GSD, Q16 Q_NMOS_GSD, Q17 Q_NMOS_GSD, Q18 Q_NMOS_GSD, Q19 Q_NMOS_GSD, Q2 Q_NMOS_GSD, Q20 Q_NMOS_GSD, Q21 Q_NMOS_GSD, Q22 Q_NMOS_GSD, Q23 Q_NMOS_GSD, Q24 NMOS, Q25 NMOS, Q26 NMOS, Q27 NMOS, Q28 NMOS, Q29 NMOS, Q3 Q_NMOS_GSD, Q30 NMOS, Q31 NMOS, Q32 NMOS, Q33 NMOS, Q34 NMOS, Q35 NMOS, Q4 Q_NMOS_GSD, Q5 Q_NMOS_GSD, Q6 Q_NMOS_GSD, Q7 Q_NMOS_GSD, Q8 Q_NMOS_GSD, Q9 Q_NMOS_GSD, SW1 SW_SPDT, SW2 SW_Push, SW3 SW_SPDT, U2 TL431DBZ, U3 TL431DBZ, U4 STM32F072RBTx, U5 SN65HVD230, U6 AP7370-33SA-7, Y1 8M,SMD, Y2 32.768k,SMD

Commit message: ready to layout pt1
Parts:
- removed C36, C37: 1u,0603, Capacitor_SMD:C_0603_1608Metric
- removed D24: GREEN_LED, LED_SMD:LED_0603_1608Metric
- removed SW1: SW_SPDT, PROYEK_BMS_NUVOTON:SW_100SP1T1B1M1QEH
- removed U6: AP7370-33SA-7, Package_TO_SOT_SMD:SOT-23-3
- added C50: 0.1u, Capacitor_SMD:C_0805_2012Metric, F.Cu at (-79.3, 113.3)
- added C51: 0.1u, Capacitor_SMD:C_0805_2012Metric, F.Cu at (-79.3, 116.3)
- added R135: NTC10k, Resistor_SMD:R_0603_1608Metric, F.Cu at (-100.9, 119.0)
- added R136: NTC10k, Resistor_SMD:R_0603_1608Metric, F.Cu at (-100.9, 121.5)
- added R137: 75M, Resistor_SMD:R_0805_2012Metric, F.Cu at (-36.1, 117.5)
- added R138: 2R2, Resistor_SMD:R_0603_1608Metric, F.Cu at (-100.9, 124.1)
- added R139: 2R2, Resistor_SMD:R_0603_1608Metric, F.Cu at (-100.9, 126.6)
- added R140: 2R2, Resistor_SMD:R_0603_1608Metric, F.Cu at (-96.9, 104.0)
- added R141: 2R2, Resistor_SMD:R_0603_1608Metric, F.Cu at (-96.9, 106.5)
- added R142: 2R2, Resistor_SMD:R_0603_1608Metric, F.Cu at (-96.9, 109.0)
- added R143: 2R2, Resistor_SMD:R_0603_1608Metric, F.Cu at (-96.9, 111.5)
- added R144: 2R2, Resistor_SMD:R_0603_1608Metric, F.Cu at (-96.9, 114.0)
- added R145: 2R2, Resistor_SMD:R_0603_1608Metric, F.Cu at (-96.9, 116.5)
- added R146: 2R2, Resistor_SMD:R_0603_1608Metric, F.Cu at (-96.9, 119.0)
- added R147: 2R2, Resistor_SMD:R_0603_1608Metric, F.Cu at (-96.9, 121.5)
- added R148: 2R2, Resistor_SMD:R_0603_1608Metric, F.Cu at (-96.9, 124.1)
- added REF**: MountingHole_5.3mm_M5_Pad, MountingHole:MountingHole_5.3mm_M5_Pad, F.Cu at (230.6, 130.2)
- added REF**: MountingHole_5.3mm_M5_Pad, MountingHole:MountingHole_5.3mm_M5_Pad, F.Cu at (212.2, 130.2)
- added U1: KA49522, Package_QFP:HTQFP-64-1EP_10x10mm_P0.5mm_EP8x8mm, F.Cu at (142.2, 73.7)
- C1: value 2.2u -> 4.7u
- C12, C3: value 100n -> 1n
- J1: footprint Connector_PinHeader_2.54mm:PinHeader_1x23_P2.54mm_Vertical -> Connector_PinSocket_2.54mm:PinSocket_1x23_P2.54mm_Vertical
- R1: value NTC10k -> 47k
- R114, R115, R116, R117, R118, R119, R120, R121, R25, R26, R27, R28, R29, R30, R31, R32, R33, R34, R35, R36, R56, R57, R58, R59, R60, R61, R62, R63, R64, R65, R66, R67, R86, R87, R88, R89, R90, R91, R92, R93, R94, R95, R96, R97: moved to B.Cu
- R132: value 1.2k,0603 -> 2R2
- R18: value R -> 47k
- R2: value 100 -> 30k
- moved D1 246.1 mm to (-92.8, 128.1)
- moved D2 246.1 mm to (-92.8, 130.7)
- moved D3 246.1 mm to (-92.8, 133.3)
- moved D4 246.1 mm to (-92.8, 135.9)
- moved D5 246.1 mm to (-92.8, 138.5)
- moved D6 246.1 mm to (-92.8, 141.0)
- moved D10 246.1 mm to (-88.8, 135.9)
- moved D11 246.1 mm to (-88.8, 138.5)
- moved D12 246.1 mm to (-88.8, 141.0)
- moved D13 246.1 mm to (-84.7, 128.1)
- moved D14 246.1 mm to (-84.7, 130.7)
- moved D15 246.1 mm to (-84.7, 133.3)
- moved D16 246.1 mm to (-84.7, 135.9)
- moved D17 246.1 mm to (-84.7, 138.5)
- moved D18 246.1 mm to (-84.7, 141.0)
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Connections:
- C11 pad 1: CN4_C0 -> C0
- C11 pad 2: C0 -> CN4_C0
- C12 pad 1: TMON1 -> TMON2
- C3 pad 1: TMON2 -> TMON1
- C4 pad 1: BMS_5V -> BMS_3.3V
- D25 pad 4: +5V -> USB_5V
- Q24 pad 2: CHG -> Net-(Q24-G)
- Q25 pad 2: CHG -> Net-(Q25-G)
- Q26 pad 2: CHG -> Net-(Q26-G)
- Q27 pad 2: CHG -> Net-(Q27-G)
- Q28 pad 2: CHG -> Net-(Q28-G)
- Q29 pad 2: CHG -> Net-(Q29-G)
- Q30 pad 2: DIS -> Net-(Q30-G)
- Q31 pad 2: DIS -> Net-(Q31-G)
- Q32 pad 2: DIS -> Net-(Q32-G)
- Q33 pad 2: DIS -> Net-(Q33-G)
- Q34 pad 2: DIS -> Net-(Q34-G)
- Q35 pad 2: DIS -> Net-(Q35-G)
- R1 pad 1: TMON2 -> TMON1
- R11 pad 1: CN4_C0 -> VPACK-
- R11 pad 2: VPACK- -> CN4_C0
- R13 pad 1: CN4_C0 -> VPACK-
- R13 pad 2: VPACK- -> CN4_C0
- R130 pad 1: CN4_C22 -> Net-(U2-K)
- R132 pad 1: CN4_C0 -> CHG
- R132 pad 2: Net-(D24-K) -> Net-(Q24-G)
- R18 pad 1: TMON1 -> TMON2
- R55 pad 1: unconnected-(R55-Pad1) -> CN4_C7
- R7 pad 1: CN4_C0 -> VPACK-
- R7 pad 2: VPACK- -> CN4_C0
- R9 pad 1: CN4_C0 -> VPACK-
- R9 pad 2: VPACK- -> CN4_C0
- U2 pad 1: CHG -> Net-(U2-K)
- U2 pad 3: CN4_C22 -> CHG
- U3 pad 1: DIS -> VPACK+
- U3 pad 3: VPACK+ -> DIS
Other:
- board outline removed

Commit message: trace 0.5
Parts:
- added C49: 0.1 uF, Capacitor_SMD:C_0805_2012Metric, F.Cu at (126.9, 86.1)
- added CVBAT1: 1uF, Capacitor_SMD:C_1206_3216Metric, F.Cu at (109.0, 72.8)
- added DVBAT1: US1M, Diode_SMD:D_SMA, F.Cu at (109.0, 65.5)
- added REF**: MountingHole_5.3mm_M5_Pad, MountingHole:MountingHole_5.3mm_M5_Pad, F.Cu at (144.1, 55.9)
- added REF**: MountingHole_3.2mm_M3_Pad_Via, MountingHole:MountingHole_3.2mm_M3_Pad_Via, F.Cu at (227.4, 49.4)
- added REF**: MountingHole_3.2mm_M3_Pad_Via, MountingHole:MountingHole_3.2mm_M3_Pad_Via, F.Cu at (63.4, 143.4)
- added REF**: MountingHole_3.2mm_M3_Pad_Via, MountingHole:MountingHole_3.2mm_M3_Pad_Via, F.Cu at (63.4, 49.4)
- added REF**: MountingHole_5.3mm_M5_Pad, MountingHole:MountingHole_5.3mm_M5_Pad, F.Cu at (191.1, 55.9)
- added REF**: MountingHole_3.2mm_M3_Pad_Via, MountingHole:MountingHole_3.2mm_M3_Pad_Via, F.Cu at (227.4, 143.4)
- added RVBAT1: 100, Resistor_SMD:R_1206_3216Metric, F.Cu at (104.4, 65.7)
- added RVBAT2: 100, Resistor_SMD:R_1206_3216Metric, F.Cu at (104.4, 72.7)
- C1: footprint Capacitor_SMD:C_1210_3225Metric -> Capacitor_SMD:C_0805_2012Metric
- J1: footprint Connector_PinSocket_2.54mm:PinSocket_1x23_P2.54mm_Vertical -> Connector_PinHeader_2.54mm:PinHeader_1x23_P2.54mm_Vertical
- SW3: footprint Button_Switch_THT:SW_CuK_OS102011MA1QN1_SPDT_Angled -> Button_Switch_SMD:SW_SPDT_PCM12
- moved R142 324.9 mm to (226.7, 79.4), turned to -90 degrees
- moved R132 317.1 mm to (214.6, 79.4), turned to -90 degrees
- moved R148 314.3 mm to (217.2, 111.8), turned to 90 degrees
- moved R138 306.7 mm to (202.6, 79.4), turned to -90 degrees
- moved R147 302.1 mm to (205.1, 111.8), turned to 90 degrees
- moved R139 295.2 mm to (190.5, 79.4), turned to -90 degrees
- moved R146 290.0 mm to (193.0, 111.8), turned to 90 degrees
- moved R145 277.9 mm to (181.0, 111.8), turned to 90 degrees
- moved R140 276.4 mm to (178.4, 79.4), turned to -90 degrees
- moved R144 265.8 mm to (168.9, 111.8), turned to 90 degrees
- moved R141 264.6 mm to (166.4, 79.4), turned to -90 degrees
- moved R136 260.3 mm to (158.1, 95.9), turned to 90 degrees
- moved C3 256.7 mm to (139.1, 122.7), turned to -90 degrees
- moved R1 253.9 mm to (141.0, 122.7), turned to -90 degrees
- moved R143 253.7 mm to (156.8, 111.8), turned to 90 degrees
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Connections:
- C1 pad 2: CN4_C0 -> GND
- C10 pad 1: CN4_C0 -> GND
- C11 pad 2: CN4_C0 -> GND
- C12 pad 2: CN4_C0 -> GND
- C19 pad 2: GNDA -> GND
- C2 pad 2: CN4_C0 -> GND
- C3 pad 2: CN4_C0 -> GND
- C38 pad 2: CN4_C0 -> GND
- C39 pad 1: CN4_C0 -> GND
- C39 pad 2: /OSC_0_IN -> /OSC_IN
- C4 pad 2: CN4_C0 -> GND
- C40 pad 2: CN4_C0 -> GND
- C41 pad 2: CN4_C0 -> GND
- C42 pad 2: CN4_C0 -> GND
- C43 pad 2: CN4_C0 -> GND
- C44 pad 2: CN4_C0 -> GND
- C45 pad 1: CN4_C0 -> GND
- C46 pad 2: CN4_C0 -> GND
- C47 pad 2: CN4_C0 -> GND
- C48 pad 2: CN4_C0 -> GND
- C5 pad 2: CN4_C0 -> GND
- C50 pad 2: CN4_C0 -> GND
- C51 pad 2: CN4_C0 -> GND
- C9 pad 1: CN4_C0 -> GND
- D23 pad 3: CN4_C0 -> GND
- D25 pad 1: CN4_C0 -> GND
- J1 pad 23: CN4_C0 -> GND
- J2 pad 1: CN4_C0 -> GND
- J3 pad 5: CN4_C0 -> GND
- Q1 pad 1: Net-(Q1-C) -> REGB
- Q1 pad 2: REGB -> Net-(Q1-C)
- Q24 pad 1: REG_SUP -> Net-(Q24-G)
- Q24 pad 2: Net-(Q24-G) -> REG_SUP
- Q25 pad 1: REG_SUP -> Net-(Q25-G)
- Q25 pad 2: Net-(Q25-G) -> REG_SUP
- Q26 pad 1: REG_SUP -> Net-(Q26-G)
- Q26 pad 2: Net-(Q26-G) -> REG_SUP
- Q27 pad 1: REG_SUP -> Net-(Q27-G)
- Q27 pad 2: Net-(Q27-G) -> REG_SUP
- Q28 pad 1: REG_SUP -> Net-(Q28-G)
- Q28 pad 2: Net-(Q28-G) -> REG_SUP
- Q29 pad 1: REG_SUP -> Net-(Q29-G)
- Q29 pad 2: Net-(Q29-G) -> REG_SUP
- Q30 pad 1: REG_SUP -> Net-(Q30-G)
- Q30 pad 2: Net-(Q30-G) -> REG_SUP
- Q31 pad 1: REG_SUP -> Net-(Q31-G)
- Q31 pad 2: Net-(Q31-G) -> REG_SUP
- Q32 pad 1: REG_SUP -> Net-(Q32-G)
- Q32 pad 2: Net-(Q32-G) -> REG_SUP
- Q33 pad 1: REG_SUP -> Net-(Q33-G)
- Q33 pad 2: Net-(Q33-G) -> REG_SUP
- Q34 pad 1: REG_SUP -> Net-(Q34-G)
- Q34 pad 2: Net-(Q34-G) -> REG_SUP
- Q35 pad 1: REG_SUP -> Net-(Q35-G)
- Q35 pad 2: Net-(Q35-G) -> REG_SUP
- Q7 pad 2: CN4_C0 -> GND
- R1 pad 2: CN4_C0 -> GND
- R10 pad 1: CN4_C0 -> GND
- R11 pad 2: CN4_C0 -> GND
- R12 pad 1: CN4_C0 -> GND
- R13 pad 2: CN4_C0 -> GND
- R130 pad 1: Net-(U2-K) -> CN4_C22
- R133 pad 2: /OSC_0_OUT -> /OSC_OUT
- R135 pad 2: CN4_C0 -> GND
- R136 pad 2: CN4_C0 -> GND
- R14 pad 1: CN4_C0 -> GND
- R18 pad 2: CN4_C0 -> GND
- R4 pad 2: CN4_C0 -> GND
- R49 pad 2: CN4_C0 -> GND
- R5 pad 1: CN4_C0 -> GND
- R6 pad 1: CN4_C0 -> GND
- R7 pad 2: CN4_C0 -> GND
- R8 pad 1: CN4_C0 -> GND
- R9 pad 2: CN4_C0 -> GND
- REF** pad 1: (no net) -> VPACK+
- REF** pad 1: (no net) -> VPACK-
- SW2 pad 1: CN4_C0 -> GND
- SW3 pad 1: CN4_C0 -> GND
- U1 pad 10: CN4_C0 -> GND
- U1 pad 16: CN4_C0 -> GND
- U1 pad 52: CN4_C0 -> GND
- U1 pad 65: CN4_C0 -> GND
- U1 pad 9: CN4_C0 -> GND
- U2 pad 1: Net-(U2-K) -> CHG
- U2 pad 3: CHG -> CN4_C22
- U3 pad 1: VPACK+ -> DIS
- U3 pad 3: DIS -> VPACK+
- U4 pad 12: CN4_C0 -> GND
- U4 pad 18: CN4_C0 -> GND
- U4 pad 31: CN4_C0 -> GND
- U4 pad 47: CN4_C0 -> GND
- U4 pad 63: CN4_C0 -> GND
- U5 pad 2: CN4_C0 -> GND
- U5 pad 8: CN4_C0 -> GND
- Y1 pad 2: /OSC_0_IN -> /OSC_IN
Routing:
- net C1: track 0.00 -> 74.5 mm
- net C21: track 0.00 -> 71.4 mm
- net C2: track 0.00 -> 67.6 mm
- net C0: track 0.00 -> 64.9 mm
- net C22: track 0.00 -> 64.5 mm
- net C3: track 0.00 -> 63.5 mm
- net C19: track 0.00 -> 60.8 mm
- net C4: track 0.00 -> 60.1 mm
- net C20: track 0.00 -> 60.0 mm
- net GND: track 0.00 -> 59.6 mm, vias 0 -> 1
- net C5: track 0.00 -> 56.6 mm
- net C6: track 0.00 -> 53.8 mm
- net C17: track 0.00 -> 53.4 mm
- net C18: track 0.00 -> 51.7 mm
- net C7: track 0.00 -> 49.7 mm
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- added copper zone on B.Cu, net CN4_C1
- added copper zone on B.Cu, net CN4_C10
- added copper zone on B.Cu, net CN4_C11
- added copper zone on B.Cu, net CN4_C12
- added copper zone on B.Cu, net CN4_C13
- added copper zone on B.Cu, net CN4_C14
- added copper zone on B.Cu, net CN4_C15
- added copper zone on B.Cu, net CN4_C16
- added copper zone on B.Cu, net CN4_C17
- added copper zone on B.Cu, net CN4_C18
- added copper zone on B.Cu, net CN4_C19
- added copper zone on B.Cu, net CN4_C2
- added copper zone on B.Cu, net CN4_C20
- added copper zone on B.Cu, net CN4_C21
- added copper zone on B.Cu, net CN4_C22
- added copper zone on F.Cu, net CN4_C22
- added copper zone on In1.Cu, net CN4_C22
- added copper zone on In2.Cu, net CN4_C22
- added copper zone on B.Cu, net CN4_C3
- added copper zone on B.Cu, net CN4_C4
- added copper zone on B.Cu, net CN4_C5
- added copper zone on B.Cu, net CN4_C6
- added copper zone on B.Cu, net CN4_C7
- added copper zone on B.Cu, net CN4_C8
- added copper zone on B.Cu, net CN4_C9
- added copper zone on F.Cu, net CN4_C9
- added copper zone on F.Cu, net GND
- added copper zone on B.Cu, net Net-(D1-K)
- added copper zone on B.Cu, net Net-(D10-K)
- added copper zone on B.Cu, net Net-(D11-K)
- added copper zone on B.Cu, net Net-(D12-K)
- added copper zone on B.Cu, net Net-(D13-K)
- added copper zone on B.Cu, net Net-(D14-K)
- added copper zone on B.Cu, net Net-(D15-K)
- added copper zone on B.Cu, net Net-(D16-K)
- added copper zone on B.Cu, net Net-(D17-K)
- added copper zone on B.Cu, net Net-(D18-K)
- added copper zone on B.Cu, net Net-(D19-K)
- added copper zone on B.Cu, net Net-(D2-K)
- added copper zone on B.Cu, net Net-(D20-K)
- added copper zone on B.Cu, net Net-(D21-K)
- added copper zone on B.Cu, net Net-(D22-K)
- added copper zone on B.Cu, net Net-(D3-K)
- added copper zone on B.Cu, net Net-(D4-K)
- added copper zone on B.Cu, net Net-(D5-K)
- added copper zone on B.Cu, net Net-(D6-K)
- added copper zone on B.Cu, net Net-(D7-K)
- added copper zone on B.Cu, net Net-(D8-K)
- added copper zone on B.Cu, net Net-(D9-K)
- added copper zone on F.Cu, net Net-(Q1-C)
- added copper zone on B.Cu, net REG_SUP
- added copper zone on F.Cu, net REG_SUP
- added copper zone on In1.Cu, net REG_SUP
- added copper zone on In2.Cu, net REG_SUP
- added copper zone on B.Cu, net VPACK+
- added copper zone on F.Cu, net VPACK+
- added copper zone on In1.Cu, net VPACK+
- added copper zone on In2.Cu, net VPACK+
- added copper zone on F.Cu, net VPACK-
Other:
- board outline added: 170 x 100 mm
- copper layers 2 -> 4

Commit message: trace 74%
Parts:
- added C36: 100n,0603, Capacitor_SMD:C_0603_1608Metric, F.Cu at (108.1, 121.3)
- added JP1: Jumper_2_Bridged, Jumper:SolderJumper-2_P1.3mm_Bridged_RoundedPad1.0x1.5mm, F.Cu at (128.3, 107.8)
- added NT1: NetTie_2, NetTie:NetTie-2_SMD_Pad0.5mm, B.Cu at (143.8, 99.1)
- added SW1: SW_Push, Button_Switch_SMD:SW_SPST_SKQG_WithStem, F.Cu at (111.8, 70.1)
- C1: footprint Capacitor_SMD:C_0805_2012Metric -> Capacitor_SMD:C_1210_3225Metric
- C50, C51, C8: footprint Capacitor_SMD:C_0805_2012Metric -> Capacitor_SMD:C_0603_1608Metric
- R3, R4: footprint Capacitor_SMD:C_0805_2012Metric_Pad1.18x1.45mm_HandSolder -> Capacitor_SMD:C_0603_1608Metric
- moved U2 69.6 mm to (191.9, 75.2), turned to 90 degrees
- moved R4 69.1 mm to (128.2, 101.9)
- moved C50 68.8 mm to (128.2, 98.7)
- moved R130 68.3 mm to (193.0, 79.4), turned to -90 degrees
- moved C8 68.1 mm to (125.6, 101.1), turned to -90 degrees
- moved R3 67.6 mm to (128.2, 100.3)
- moved C51 66.9 mm to (128.2, 103.6)
- moved U3 66.0 mm to (191.8, 115.6), turned to -90 degrees
- moved R131 64.6 mm to (190.8, 111.6), turned to 90 degrees
- moved C45 21.2 mm to (123.0, 127.7), turned to 180 degrees
- moved R134 14.7 mm to (126.9, 132.2), turned to 180 degrees
- moved C5 13.8 mm to (112.9, 78.0), turned to 90 degrees
- moved U5 11.3 mm to (108.1, 125.7)
- moved C46 10.3 mm to (123.0, 125.7), turned to 0 degrees
- moved Y2 9.62 mm to (116.9, 126.7)
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Connections:
- J4 pad 1: /CAN_D+ -> /CAN_D-
- J4 pad 2: /CAN_D- -> /CAN_D+
- R4 pad 2: GND -> Net-(NT1-Pad2)
- U4 pad 3: /OSC32_OUT -> /OSC32_IN
- Y2 pad 2: /OSC32_IN -> unconnected-(Y2-Pad2)
- Y2 pad 3: (no net) -> unconnected-(Y2-Pad3)
- Y2 pad 4: (no net) -> /OSC32_IN
Routing:
- net DIS: track 0.00 -> 187.3 mm, vias 0 -> 2
- net CHG: track 0.00 -> 185.5 mm, vias 0 -> 2
- net GND: track 59.6 -> 203.7 mm, vias 1 -> 145
- net TMON1: track 0.00 -> 51.1 mm, vias 0 -> 2
- net TMON2: track 0.00 -> 42.5 mm, vias 0 -> 4
- net /OSC32_IN: track 0.00 -> 40.8 mm
- net +3V3: track 0.00 -> 39.0 mm, vias 0 -> 12
- net BMS_3.3V: track 0.00 -> 38.9 mm, vias 0 -> 4
- net /USB_D-: track 0.00 -> 38.8 mm
- net /RESET: track 0.00 -> 38.8 mm
- net VPACK+: track 0.00 -> 38.7 mm, vias 0 -> 70
- net /OSC32_OUT: track 0.00 -> 38.1 mm
- net /USB_D+: track 0.00 -> 37.5 mm
- net SHDN: track 0.00 -> 34.5 mm, vias 0 -> 2
- net REGB: track 0.00 -> 33.1 mm, vias 0 -> 2
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- added copper zone on F.Cu, net +3V3
- added copper zone on In2.Cu, net +3V3
- added copper zone on B.Cu, net GND
- added copper zone on In1.Cu, net GND
- added copper zone on B.Cu, net Net-(Q1-C)
- added copper zone on In1.Cu, net Net-(Q1-C)
- added copper zone on In2.Cu, net Net-(Q1-C)
- added copper zone on In1.Cu, net VPACK-
