File: PROYEK_BMS_NUVOTON.kicad_sch (KiCad schematic)
At the start: 268 parts, among them J1 Conn_01x23_Pin, J2 Conn_01x04_Pin, J3 USB_B_Micro, J4 Screw_Terminal_01x02, Q1 NPN, Q17 Q_NMOS_GSD, Q18 Q_NMOS_GSD, Q19 Q_NMOS_GSD, Q20 Q_NMOS_GSD, Q21 Q_NMOS_GSD, Q22 Q_NMOS_GSD, Q23 Q_NMOS_GSD, Q24 Q_NMOS_GSD, Q25 Q_NMOS_GSD, Q26 Q_NMOS_GSD, Q27 Q_NMOS_GSD, Q28 Q_NMOS_GSD, Q29 Q_NMOS_GSD, Q30 Q_NMOS_GSD, Q31 Q_NMOS_GSD, Q32 Q_NMOS_GSD, Q33 Q_NMOS_GSD, Q34 Q_NMOS_GSD, Q35 Q_NMOS_GSD, Q36 Q_NMOS_GSD, Q37 Q_NMOS_GSD, Q38 Q_NMOS_GSD, Q5 NMOS, Q6 NMOS, SW1 SW_SPDT, SW2 SW_Push, SW3 SW_SPDT, SW4 SW_Push, U1 KA49522, U2 TL431DBZ, U4 STM32F072RBTx, U5 SN65HVD230, U6 AP7370-33SA-7, Y1 8M,SMD, Y2 32.768k,SMD

Commit message: ready to layout pt1
Parts:
- removed C36, C37: 1u,0603, Capacitor_SMD:C_0603_1608Metric, symbol Device:C
- removed D24: GREEN_LED, LED_SMD:LED_0603_1608Metric, symbol Device:LED
- removed Q5 (x7), Q6 (x4): NMOS, Package_TO_SOT_SMD:TO-263-2, symbol Simulation_SPICE:NMOS
- removed SW1: SW_SPDT, PROYEK_BMS_NUVOTON:SW_100SP1T1B1M1QEH, symbol Switch:SW_SPDT
- removed U6: AP7370-33SA-7, Package_TO_SOT_SMD:SOT-23-3, symbol Regulator_Linear:AP7370-33FDC
- added Q6 (x11): NMOS, Package_TO_SOT_SMD:TO-263-2, symbol Simulation_SPICE:NMOS
- added R138, R139, R140, R141, R142, R143, R144, R145, R146, R147, R148: 2R2, Resistor_SMD:R_0603_1608Metric, symbol Device:R
- R132: value 1.2k,0603 -> 2R2; JLCPCB Part # C22765 -> C25810
Connections:
- net +5V is gone; now on net USB_5V: D25.4 (VCC)
- net CHG: now also R132.1, R138.1, R139.1, R140.1, R141.1, R142.1; no longer Q6.2 (G)
- net CN4_C22: now also Q6.3 (S), Q6.3 (S), Q6.3 (S), Q6.3 (S), Q6.3 (S); no longer CVBAT1.2, RVBAT2.2, U1.28 (VBAT)
- net DIS: now also R143.1, R144.1, R145.1, R146.1, R147.1, R148.1
- net GND: no longer R132.1
- net REG_SUP: now also Q6.1 (D), Q6.1 (D), Q6.1 (D), Q6.1 (D), Q6.1 (D), Q6.1 (D), Q6.1 (D), Q6.1 (D), Q6.1 (D), Q6.1 (D), Q6.1 (D)
- net VPACK+: now also Q6.3 (S), Q6.3 (S), Q6.3 (S), Q6.3 (S), Q6.3 (S), Q6.3 (S)
- net at R132.2: now also Q6.2 (G)
- new net: Q6.2 (G), R145.2
- new net: Q6.2 (G), R147.2
- new net: Q6.2 (G), R138.2
- new net: Q6.2 (G), R139.2
- new net: Q6.2 (G), R148.2
- new net: Q6.2 (G), R144.2
- new net: Q6.2 (G), R143.2
- new net: Q6.2 (G), R146.2
- new net: Q6.2 (G), R140.2
- new net: Q6.2 (G), R142.2
- new net: Q6.2 (G), R141.2
- new net VBAT-P: CVBAT1.2, RVBAT2.2, U1.28 (VBAT)
Other:
- moved on the sheet: D23, Q6, R75, R76, U2

Commit message: trace 0.5
Parts:
- added C36: 100n,0603, Capacitor_SMD:C_0603_1608Metric, symbol Device:C
- added JP1: Jumper_2_Bridged, symbol Jumper:Jumper_2_Bridged
- C49: footprint (none) -> Capacitor_SMD:C_0805_2012Metric
- CVBAT1: footprint (none) -> Capacitor_SMD:C_1206_3216Metric
- DVBAT1: value NHP120SFT3G -> US1M; footprint (none) -> Diode_SMD:D_SMA; JLCPCB Part # (none) -> C412437
- J1: footprint (none) -> Connector_PinHeader_2.54mm:PinHeader_1x23_P2.54mm_Vertical
- Q1: symbol Simulation_SPICE:NPN -> Device:Q_NPN_BCE
- Q6: symbol Simulation_SPICE:NMOS -> Device:Q_NMOS_GDS
- RVBAT1, RVBAT2: footprint (none) -> Resistor_SMD:R_1206_3216Metric
- SW3: footprint Button_Switch_THT:SW_CuK_OS102011MA1QN1_SPDT_Angled -> Button_Switch_SMD:SW_SPDT_PCM12
- U1: footprint Package_QFP:HTQFP-64-1EP_10x10mm_P0.5mm_EP5.5x5.5mm_Mask4.4x4.4mm_ThermalVias -> Package_QFP:HTQFP-64-1EP_10x10mm_P0.5mm_EP8x8mm
- Y2: symbol Device:Crystal -> Device:Crystal_GND23
Connections:
- net GNDA is gone; now on net GND: C67.2, CVBAT1.1
- net OSC_0_IN is gone; now on net OSC_IN: C39.2, Y1.2
- net OSC_0_OUT is gone; now on net OSC_OUT: R133.2
- net +3V3: now also C36.1, JP1.2 (B)
- net BMS_3.3V: now also JP1.1 (A)
- net CAN_D+: now also J4.2 (Pin_2); no longer J4.1 (Pin_1)
- net CAN_D-: now also J4.1 (Pin_1); no longer J4.2 (Pin_2)
- net GND: now also C36.2
- net OSC32_IN: now also U4.3 (PC14), Y2.4; no longer Y2.2
- net OSC32_OUT: no longer U4.3 (PC14)
- net REGB: now also Q1.1 (B); no longer Q1.2 (B)
- net REG_SUP: now also Q6.2 (D), Q6.2 (D), Q6.2 (D), Q6.2 (D), Q6.2 (D), Q6.2 (D), Q6.2 (D), Q6.2 (D), Q6.2 (D), Q6.2 (D), Q6.2 (D), Q6.2 (D); no longer Q6.1 (D), Q6.1 (D), Q6.1 (D), Q6.1 (D), Q6.1 (D), Q6.1 (D), Q6.1 (D), Q6.1 (D), Q6.1 (D), Q6.1 (D), Q6.1 (D), Q6.1 (D)
- net at R145.2: now also Q6.1 (G); no longer Q6.2 (G)
- net at R147.2: now also Q6.1 (G); no longer Q6.2 (G)
- net at R138.2: now also Q6.1 (G); no longer Q6.2 (G)
- net at R139.2: now also Q6.1 (G); no longer Q6.2 (G)
- net at R148.2: now also Q6.1 (G); no longer Q6.2 (G)
- net at R132.2: now also Q6.1 (G); no longer Q6.2 (G)
- net at R15.2: now also Q1.2 (C); no longer Q1.1 (C)
- net at R144.2: now also Q6.1 (G); no longer Q6.2 (G)
- net at R143.2: now also Q6.1 (G); no longer Q6.2 (G)
- net at R146.2: now also Q6.1 (G); no longer Q6.2 (G)
- net at R140.2: now also Q6.1 (G); no longer Q6.2 (G)
- net at R142.2: now also Q6.1 (G); no longer Q6.2 (G)
- net at R141.2: now also Q6.1 (G); no longer Q6.2 (G)
Other:
- moved on the sheet: SW4

Commit message: trace 74%
Parts:
- removed SW4: SW_Push, symbol Switch:SW_Push
- added NT1: NetTie_2, NetTie:NetTie-2_SMD_Pad0.5mm, symbol Device:NetTie_2
- added SW1: SW_Push, Button_Switch_SMD:SW_SPST_SKQG_WithStem, symbol Switch:SW_Push
- C23: footprint Capacitor_SMD:C_0805_2012Metric -> Capacitor_SMD:C_0603_1608Metric
- JP1: footprint (none) -> Jumper:SolderJumper-2_P1.3mm_Bridged_RoundedPad1.0x1.5mm
- R25, R26: footprint Capacitor_SMD:C_0805_2012Metric_Pad1.18x1.45mm_HandSolder -> Capacitor_SMD:C_0603_1608Metric
Connections:
- net GND: now also NT1.1; no longer R25.2
- net VPACK+: now also SW1.2
- net at R137.1: now also SW1.1
- new net: NT1.2, R25.2
Changed lines of the file:
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@@
     (stroke (width 0) (type default))
   )
+  (wire (pts (xy 135.89 408.94) (xy 135.89 411.48))
+    (stroke (width 0) (type default))
+  )
   (wire (pts (xy 127 262.89) (xy 130.81 262.89))
     (stroke (width 0) (type default))
@@
     (stroke (width 0) (type default))
   )
-  (wire (pts (xy 135.89 416.56) (xy 135.89 408.94))
-    (stroke (width 0) (type default))
-  )
   (wire (pts (xy 285.75 363.22) (xy 285.75 364.49))
     (stroke (width 0) (type default))
@@
     (stroke (width 0) (type default))
   )
-  (wire (pts (xy 140.97 410.21) (xy 140.97 408.94))
+  (wire (pts (xy 143.51 410.21) (xy 143.51 408.94))
     (stroke (width 0) (type default))
   )
@@
     (stroke (width 0) (type default))
   )
-  (wire (pts (xy 140.97 408.94) (xy 135.89 408.94))
+  (wire (pts (xy 143.51 408.94) (xy 135.89 408.94))
     (stroke (width 0) (type default))
   )
@@
       (effects (font (size 1.27 1.27)))
     )
-    (property "Footprint" "Capacitor_SMD:C_0805_2012Metric" (at 124.1552 443.23 0)
+    (property "Footprint" "Capacitor_SMD:C_0603_1608Metric" (at 124.1552 443.23 0)
       (effects (font (size 1.27 1.27)) hide)
     )
@@
       (effects (font (size 1.27 1.27)))
     )
-    (property "Footprint" "" (at 604.52 462.28 0)
+    (property "Footprint" "Jumper:SolderJumper-2_P1.3mm_Bridged_RoundedPad1.0x1.5mm" (at 604.52 462.28 0)
       (effects (font (size 1.27 1.27)) hide)
     )
@@
       (effects (font (size 1.27 1.27)))
     )
-    (property "Footprint" "Capacitor_SMD:C_0805_2012Metric" (at 137.4648 443.23 0)
+    (property "Footprint" "Capacitor_SMD:C_0603_1608Metric" (at 137.4648 443.23 0)
       (effects (font (size 1.27 1.27)) hide)
     )
@@
       (effects (font (size 1.27 1.27)))
     )
-    (property "Footprint" "Capacitor_SMD:C_0805_2012Metric" (at 134.62 428.2948 0)
+    (property "Footprint" "Capacitor_SMD:C_0603_1608Metric" (at 134.62 428.2948 0)
       (effects (font (size 1.27 1.27)) hide)
     )
@@
     )
   )
+  (symbol (lib_id "Device:NetTie_2") (at 135.89 414.02 270) (unit 1)
+    (in_bom no) (on_board yes) (dnp no)
+    (property "Reference" "NT1" (at 137.16 414.02 90)
+      (effects (font (size 1.27 1.27)) (justify left))
+    )
+    (property "Value" "NetTie_2" (at 137.16 415.29 90)
+      (effects (font (size 1.27 1.27)) (justify left) hide)
+    )
+    (property "Footprint" "NetTie:NetTie-2_SMD_Pad0.5mm" (at 135.89 414.02 0)
+      (effects (font (size 1.27 1.27)) hide)
+    )
+    (property "Datasheet" "~" (at 135.89 414.02 0)
+      (effects (font (size 1.27 1.27)) hide)
+    )
+    (pin "1")
+    (pin "2")
+    (instances
+      (project "PROYEK_BMS_NUVOTON"
+        (path "/61bf283a-d7f5-4326-b612-ca4160d295db"
+          (reference "NT1") (unit 1)
+        )
+      )
+    )
+  )
   (symbol (lib_id "Device:R") (at 130.81 368.3 90) (mirror x) (unit 1)
     (in_bom yes) (on_board yes) (dnp no)
@@
       (effects (font (size 1.27 1.27)) (justify left))
     )
-    (property "Footprint" "Capacitor_SMD:C_0805_2012Metric_Pad1.18x1.45mm_HandSolder" (at 134.112 420.37 90)
+    (property "Footprint" "Capacitor_SMD:C_0603_1608Metric" (at 134.112 420.37 90)
       (effects (font (size 1.27 1.27)) hide)
     )
@@
     )
   )
+  (symbol (lib_id "Switch:SW_Push") (at 190.5 36.83 90) (unit 1)
+    (in_bom yes) (on_board yes) (dnp no)
+    (property "Reference" "SW1" (at 198.12 35.56 90)
+      (effects (font (size 1.27 1.27)) (justify right))
+    )
+    (property "Value" "SW_Push" (at 198.12 38.1 90)
+      (effects (font (size 1.27 1.27)) (justify right))
+    )
+    (property "Footprint" "Button_Switch_SMD:SW_SPST_SKQG_WithStem" (at 185.42 36.83 0)
+      (effects (font (size 1.27 1.27)) hide)
+    )
+    (property "Datasheet" "~" (at 185.42 36.83 0)
+      (effects (font (size 1.27 1.27)) hide)
+    )
+    (property "JLCPCB Part #" "C318884" (at 190.5 36.83 0)
+      (effects (font (size 1.27 1.27)) hide)
+    )
+    (pin "1")
+    (pin "2")
+    (instances
+      (project "PROYEK_BMS_NUVOTON"
+        (path "/61bf283a-d7f5-4326-b612-ca4160d295db"
+          (reference "SW1") (unit 1)
+        )
+      )
+      (project "board_bms"
+        (path "/9f5383c6-2629-4a7d-b7b2-5028aa228484"
+          (reference "SW1") (unit 1)
+        )
+      )
+    )
+  )
   (symbol (lib_id "MCU_ST_STM32F0:STM32F072RBTx") (at 523.24 407.67 0) (unit 1)
     (in_bom yes) (on_board yes) (dnp no) (fields_autoplaced)
@@
       (effects (font (size 1.27 1.27)) (justify left))
     )
-    (property "Footprint" "Capacitor_SMD:C_0805_2012Metric_Pad1.18x1.45mm_HandSolder" (at 127.508 420.37 90)
+    (property "Footprint" "Capacitor_SMD:C_0603_1608Metric" (at 127.508 420.37 90)
       (effects (font (size 1.27 1.27)) hide)
     )
@@
     )
   )
-  (symbol (lib_id "Switch:SW_Push") (at 190.5 36.83 270) (mirror x) (unit 1)
-    (in_bom yes) (on_board yes) (dnp no)
-    (property "Reference" "SW4" (at 189.23 35.56 90)
-      (effects (font (size 1.27 1.27)) (justify right))
-    )
-    (property "Value" "SW_Push" (at 189.23 38.1 90)
-      (effects (font (size 1.27 1.27)) (justify right))
-    )
-    (property "Footprint" "" (at 195.58 36.83 0)
-      (effects (font (size 1.27 1.27)) hide)
-    )
-    (property "Datasheet" "~" (at 195.58 36.83 0)
-      (effects (font (size 1.27 1.27)) hide)
-    )
-    (pin "1")
-    (pin "2")
-    (instances
-      (project "PROYEK_BMS_NUVOTON"
-        (path "/61bf283a-d7f5-4326-b612-ca4160d295db"
-          (reference "SW4") (unit 1)
-        )
-      )
-    )
-  )
   (symbol (lib_id "Device:Q_NMOS_GSD") (at 231.14 510.54 0) (mirror y) (unit 1)
     (in_bom yes) (on_board yes) (dnp no) (fields_autoplaced)
@@
     )
   )
-  (symbol (lib_id "power:GND") (at 140.97 410.21 0) (unit 1)
+  (symbol (lib_id "power:GND") (at 143.51 410.21 0) (unit 1)
     (in_bom yes) (on_board yes) (dnp no) (fields_autoplaced)
-    (property "Reference" "#PWR011" (at 140.97 416.56 0)
+    (property "Reference" "#PWR011" (at 143.51 416.56 0)
       (effects (font (size 1.27 1.27)) hide)
     )
-    (property "Value" "GND" (at 144.78 411.48 0)
+    (property "Value" "GND" (at 147.32 411.48 0)
       (effects (font (size 1.27 1.27)) (justify left))
     )
-    (property "Footprint" "" (at 140.97 410.21 0)
+    (property "Footprint" "" (at 143.51 410.21 0)
       (effects (font (size 1.27 1.27)) hide)
     )
-    (property "Datasheet" "" (at 140.97 410.21 0)
+    (property "Datasheet" "" (at 143.51 410.21 0)
       (effects (font (size 1.27 1.27)) hide)
     )
